File: Harley/HarleyProcessing/HarleyProcessing.kicad_pcb (KiCad board)
At the start: 2 copper layers, 30 x 31 mm, 55 parts, among them P2 CONN_02X40, P3 CONN_02X40, P4 CONN_02X40, U1 xc7a50tcsg324pkg, U2 LTM4622, U3 MT41K128M16, U4 LTM4622, U5 OSCILLATOR, U6 OSCILLATOR

Commit message: starting placing passives for HarleyFullMC
Parts:
- U3: footprint BGA:WBGA96C80P6X16_90X1300X120 -> BGA:WBGA96C80P6X16_80X1400X110
Changed lines of the file:
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@@
     )
   )
-  (module BGA:WBGA96C80P6X16_90X1300X120 (layer F.Cu)
+  (module Mounting:MountingHoleM1.6 (layer F.Cu)
+    (at 13.5 196.5)
+    (descr "MountingHole M1.6 screws")
+    (tags "M1.6 Mount Hole")
+    (fp_text reference REF** (at 0.1 4.4) (layer F.SilkS) hide
+      (effects (font (size 1 1) (thickness 0.15)))
+    )
+    (fp_text value MountingHoleM2 (at 0 -4) (layer F.Fab)
+      (effects (font (size 1 1) (thickness 0.15)))
+    )
+    (fp_circle (center 0 0) (end -1.5 0) (layer F.SilkS) (width 0.15))
+    (fp_circle (center 0 0) (end -1.6 0) (layer F.CrtYd) (width 0.05))
+    (fp_circle (center 0 0) (end -1.1 -1.1) (layer B.CrtYd) (width 0.05))
+    (pad MNT thru_hole circle (at 0 0) (size 2.2 2.2) (drill 1.8) (layers *.Cu *.Mask F.SilkS))
+  )
+  (module Mounting:MountingHoleM1.6 (layer F.Cu)
+    (at 40.5 196.5)
+    (descr "MountingHole M1.6 screws")
+    (tags "M1.6 Mount Hole")
+    (fp_text reference REF** (at 0.1 4.4) (layer F.SilkS) hide
+      (effects (font (size 1 1) (thickness 0.15)))
+    )
+    (fp_text value MountingHoleM2 (at 0 -4) (layer F.Fab)
+      (effects (font (size 1 1) (thickness 0.15)))
+    )
+    (fp_circle (center 0 0) (end -1.5 0) (layer F.SilkS) (width 0.15))
+    (fp_circle (center 0 0) (end -1.6 0) (layer F.CrtYd) (width 0.05))
+    (fp_circle (center 0 0) (end -1.1 -1.1) (layer B.CrtYd) (width 0.05))
+    (pad MNT thru_hole circle (at 0 0) (size 2.2 2.2) (drill 1.8) (layers *.Cu *.Mask F.SilkS))
+  )
+  (module Mounting:MountingHoleM1.6 (layer F.Cu)
+    (at 40.5 168.5)
+    (descr "MountingHole M1.6 screws")
+    (tags "M1.6 Mount Hole")
+    (fp_text reference REF** (at 0.1 4.4) (layer F.SilkS) hide
+      (effects (font (size 1 1) (thickness 0.15)))
+    )
+    (fp_text value MountingHoleM2 (at 0 -4) (layer F.Fab)
+      (effects (font (size 1 1) (thickness 0.15)))
+    )
+    (fp_circle (center 0 0) (end -1.5 0) (layer F.SilkS) (width 0.15))
+    (fp_circle (center 0 0) (end -1.6 0) (layer F.CrtYd) (width 0.05))
+    (fp_circle (center 0 0) (end -1.1 -1.1) (layer B.CrtYd) (width 0.05))
+    (pad MNT thru_hole circle (at 0 0) (size 2.2 2.2) (drill 1.8) (layers *.Cu *.Mask F.SilkS))
+  )
+  (module Mounting:MountingHoleM1.6 (layer F.Cu)
+    (at 13.5 168.5)
+    (descr "MountingHole M1.6 screws")
+    (tags "M1.6 Mount Hole")
+    (fp_text reference REF** (at 0.1 4.4) (layer F.SilkS) hide
+      (effects (font (size 1 1) (thickness 0.15)))
+    )
+    (fp_text value MountingHoleM2 (at 0 -4) (layer F.Fab)
+      (effects (font (size 1 1) (thickness 0.15)))
+    )
+    (fp_circle (center 0 0) (end -1.5 0) (layer F.SilkS) (width 0.15))
+    (fp_circle (center 0 0) (end -1.6 0) (layer F.CrtYd) (width 0.05))
+    (fp_circle (center 0 0) (end -1.1 -1.1) (layer B.CrtYd) (width 0.05))
+    (pad MNT thru_hole circle (at 0 0) (size 2.2 2.2) (drill 1.8) (layers *.Cu *.Mask F.SilkS))
+  )
+  (module BGA:WBGA96C80P6X16_80X1400X110 (layer F.Cu)
     (at 26.9 173 90)
     (descr "WBGA96 with 3 empty column ")
@@
     (pad T9 smd circle (at 3.2 6 90) (size 0.4 0.4) (layers F.Cu F.Paste F.Mask)
       (net 547 GND))
-    (model /home/mikael/work/kicad_ws/osrf_hw_nonfree/BGA.3dshapes/WBGA96C80P6X16_90X1300X120.wrl
+    (model /home/mikael/work/kicad_ws/osrf_hw_nonfree/BGA.3dshapes/WBGA96C80P6X16_80X1400X110.wrl
       (at (xyz 0 0 0))
       (scale (xyz 1 1 1))
@@
     )
   )
-  (module Mounting:MountingHoleM1.6 (layer F.Cu)
-    (at 13.5 196.5)
-    (descr "MountingHole M1.6 screws")
-    (tags "M1.6 Mount Hole")
-    (fp_text reference REF** (at 0.1 4.4) (layer F.SilkS) hide
-      (effects (font (size 1 1) (thickness 0.15)))
-    )
-    (fp_text value MountingHoleM2 (at 0 -4) (layer F.Fab)
-      (effects (font (size 1 1) (thickness 0.15)))
-    )
-    (fp_circle (center 0 0) (end -1.5 0) (layer F.SilkS) (width 0.15))
-    (fp_circle (center 0 0) (end -1.6 0) (layer F.CrtYd) (width 0.05))
-    (fp_circle (center 0 0) (end -1.1 -1.1) (layer B.CrtYd) (width 0.05))
-    (pad MNT thru_hole circle (at 0 0) (size 2.2 2.2) (drill 1.8) (layers *.Cu *.Mask F.SilkS))
-  )
-  (module Mounting:MountingHoleM1.6 (layer F.Cu)
-    (at 40.5 196.5)
-    (descr "MountingHole M1.6 screws")
-    (tags "M1.6 Mount Hole")
-    (fp_text reference REF** (at 0.1 4.4) (layer F.SilkS) hide
-      (effects (font (size 1 1) (thickness 0.15)))
-    )
-    (fp_text value MountingHoleM2 (at 0 -4) (layer F.Fab)
-      (effects (font (size 1 1) (thickness 0.15)))
-    )
-    (fp_circle (center 0 0) (end -1.5 0) (layer F.SilkS) (width 0.15))
-    (fp_circle (center 0 0) (end -1.6 0) (layer F.CrtYd) (width 0.05))
-    (fp_circle (center 0 0) (end -1.1 -1.1) (layer B.CrtYd) (width 0.05))
-    (pad MNT thru_hole circle (at 0 0) (size 2.2 2.2) (drill 1.8) (layers *.Cu *.Mask F.SilkS))
-  )
-  (module Mounting:MountingHoleM1.6 (layer F.Cu)
-    (at 40.5 168.5)
-    (descr "MountingHole M1.6 screws")
-    (tags "M1.6 Mount Hole")
-    (fp_text reference REF** (at 0.1 4.4) (layer F.SilkS) hide
-      (effects (font (size 1 1) (thickness 0.15)))
-    )
-    (fp_text value MountingHoleM2 (at 0 -4) (layer F.Fab)
-      (effects (font (size 1 1) (thickness 0.15)))
-    )
-    (fp_circle (center 0 0) (end -1.5 0) (layer F.SilkS) (width 0.15))
-    (fp_circle (center 0 0) (end -1.6 0) (layer F.CrtYd) (width 0.05))
-    (fp_circle (center 0 0) (end -1.1 -1.1) (layer B.CrtYd) (width 0.05))
-    (pad MNT thru_hole circle (at 0 0) (size 2.2 2.2) (drill 1.8) (layers *.Cu *.Mask F.SilkS))
-  )
-  (module Mounting:MountingHoleM1.6 (layer F.Cu)
-    (at 13.5 168.5)
-    (descr "MountingHole M1.6 screws")
-    (tags "M1.6 Mount Hole")
-    (fp_text reference REF** (at 0.1 4.4) (layer F.SilkS) hide
-      (effects (font (size 1 1) (thickness 0.15)))
-    )
-    (fp_text value MountingHoleM2 (at 0 -4) (layer F.Fab)
-      (effects (font (size 1 1) (thickness 0.15)))
-    )
-    (fp_circle (center 0 0) (end -1.5 0) (layer F.SilkS) (width 0.15))
-    (fp_circle (center 0 0) (end -1.6 0) (layer F.CrtYd) (width 0.05))
-    (fp_circle (center 0 0) (end -1.1 -1.1) (layer B.CrtYd) (width 0.05))
-    (pad MNT thru_hole circle (at 0 0) (size 2.2 2.2) (drill 1.8) (layers *.Cu *.Mask F.SilkS))
-  )
   (gr_line (start 42 198) (end 12 198) (layer Edge.Cuts) (width 0.15))
