File: hardware/ovc2/mono/ovc2_mono.kicad_pcb (KiCad board)
At the start: 6 copper layers, 87 x 55.5 mm, 137 parts, among them J16 FPGA CONFIG, J2 Conn_02x20_Odd_Even, J5 IMU DEBUG, J8 LENS_HOLDER, Q11 NTR4003NT1G, Q12 NTR4003NT1G, Q13 NTR4003NT1G, Q14 NTS4001NT1G, Q15 NTR4003NT1G, Q3 DMN2041L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

Commit message: lots of hacking
Parts:
- removed J5: IMU DEBUG, Pin_Headers:Pin_Header_Straight_1x03_Pitch2.54mm
- removed U4: VN-100, IMU:VN-100
- added Z2: Logo_Open_Hardware_Small, Symbols:OSHW-Symbol_6.7x6mm_SilkScreen, F.Cu at (138.5, 92.5)
Routing:
- net +12V: vias 10 -> 9
- net (no net): vias 3 -> 4
