File: hardware/ovc3b/camera/imagers.sch (KiCad schematic (older format))
At the start: 55 parts, among them J1 LEFT_LENS, J11 CAM2_TIMING_DEBUG, J2 RIGHT_LENS, J4 MIDDLE_LENS, U1 AR0144CS, U10 LP5907MFX-2.8, U12 LP5907MFX-2.8, U2 AR0144CS, U4 AR0144CS

Commit message: update part numbers
Parts:
- C26, C27, C28, C29, C30, C31, C36, C37, C38, C39, C40, C41, C44, C47, C48, C49, C50, C51, C54, C55, C56, C57, C58, C59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: D1PN 1276-1004-1-ND -> 490-11917-1-ND; MFN Samsung -> Murata; MPN CL05F104ZO5NNNC -> GRM155R61H104KE19D
