File: hardware/ovc3b/camera/imu.sch (KiCad schematic (older format))
At the start: 4 parts, among them U3 ICM-20948

Commit message: update part numbers
Parts:
- C11, C12, C13: D1PN 1276-1004-1-ND -> 490-11917-1-ND; MFN Samsung -> Murata; MPN CL05F104ZO5NNNC -> GRM155R61H104KE19D
- U3: D1 Mouser -> Digikey; D1PN 410-ICM-20948 -> 1428-1123-1-ND
Changed lines of the file:
@@
 F 4 "Digikey" H 3892 1496 50  0001 C CNN "D1"
 F 5 "Digikey" H 3892 1496 50  0001 C CNN "D1N"
-F 6 "1276-1004-1-ND" H 3892 1496 50  0001 C CNN "D1PN"
-F 7 "Samsung" H 3892 1496 50  0001 C CNN "MFN"
-F 8 "CL05F104ZO5NNNC" H 3892 1496 50  0001 C CNN "MPN"
+F 6 "490-11917-1-ND" H 3892 1496 50  0001 C CNN "D1PN"
+F 7 "Murata" H 3892 1496 50  0001 C CNN "MFN"
+F 8 "GRM155R61H104KE19D" H 3892 1496 50  0001 C CNN "MPN"
 	1    3800 1350
 	1    0    0    -1
@@
 F 4 "Digikey" H 4692 1496 50  0001 C CNN "D1"
 F 5 "Digikey" H 4692 1496 50  0001 C CNN "D1N"
-F 6 "1276-1004-1-ND" H 4692 1496 50  0001 C CNN "D1PN"
-F 7 "Samsung" H 4692 1496 50  0001 C CNN "MFN"
-F 8 "CL05F104ZO5NNNC" H 4692 1496 50  0001 C CNN "MPN"
+F 6 "490-11917-1-ND" H 4692 1496 50  0001 C CNN "D1PN"
+F 7 "Murata" H 4692 1496 50  0001 C CNN "MFN"
+F 8 "GRM155R61H104KE19D" H 4692 1496 50  0001 C CNN "MPN"
 	1    4600 1350
 	1    0    0    -1
@@
 F 4 "Digikey" H 5342 2896 50  0001 C CNN "D1"
 F 5 "Digikey" H 5342 2896 50  0001 C CNN "D1N"
-F 6 "1276-1004-1-ND" H 5342 2896 50  0001 C CNN "D1PN"
-F 7 "Samsung" H 5342 2896 50  0001 C CNN "MFN"
-F 8 "CL05F104ZO5NNNC" H 5342 2896 50  0001 C CNN "MPN"
+F 6 "490-11917-1-ND" H 5342 2896 50  0001 C CNN "D1PN"
+F 7 "Murata" H 5342 2896 50  0001 C CNN "MFN"
+F 8 "GRM155R61H104KE19D" H 5342 2896 50  0001 C CNN "MPN"
 	1    5250 2750
 	1    0    0    -1
@@
 F 2 "Sensor_Motion:InvenSense_QFN-24_3x3mm_P0.4mm" H 4200 1450 50  0001 C CNN
 F 3 "https://store.invensense.com/datasheets/invensense/MPU9250REV1.0.pdf" H 4200 2300 50  0001 C CNN
-F 4 "Mouser" H 3800 1900 50  0001 C CNN "D1"
+F 4 "Digikey" H 3800 1900 50  0001 C CNN "D1"
 F 5 "Digikey" H 3800 1900 50  0001 C CNN "D1N"
-F 6 "410-ICM-20948" H 3800 1900 50  0001 C CNN "D1PN"
+F 6 "1428-1123-1-ND" H 3800 1900 50  0001 C CNN "D1PN"
 F 7 "TDK InvenSense" H 3800 1900 50  0001 C CNN "MFN"
 F 8 "ICM-20948" H 3800 1900 50  0001 C CNN "MPN"
