File: hardware/ovc3b/camera/te0820.sch (KiCad schematic (older format))
At the start: 32 parts, among them J12 AUX, M1 TE0820, SW1 SW_DIP_x04, U16 SN74AXCH8T245, U17 TCA9803, U18 TCA9803, U8 SN74AXC4T245

Commit message: move sdio level shifter to top side. migrate aux header towards west side.
Parts:
- removed J12: AUX, Connector_PinHeader_1.27mm:PinHeader_2x04_P1.27mm_Vertical, symbol Connector_Generic:Conn_02x04_Odd_Even
Connections:
- net labels added: LED2, LED3
- wire segments 208 -> 206
Other:
- note added: "TODO: assign "AUX" pins to north bonus header"
Changed lines of the file:
@@
-	1    0    0    -1
-$EndComp
-$Comp
-L power:GND #PWR0111
-U 1 1 5CB44C25
-P 3600 7000
-F 0 "#PWR0111" H 3600 6750 50  0001 C CNN
-F 1 "GND" H 3605 6827 50  0001 C CNN
-F 2 "" H 3600 7000 50  0001 C CNN
-F 3 "" H 3600 7000 50  0001 C CNN
-	1    3600 7000
-	1    0    0    -1
-$EndComp
-$Comp
-L Connector_Generic:Conn_02x04_Odd_Even J12
-U 1 1 5CB74256
-P 2900 6900
-F 0 "J12" H 2950 7217 50  0000 C CNN
-F 1 "AUX" H 2950 7126 50  0000 C CNN
-F 2 "Connector_PinHeader_1.27mm:PinHeader_2x04_P1.27mm_Vertical" H 2900 6900 50  0001 C CNN
-F 3 "~" H 2900 6900 50  0001 C CNN
-F 4 "DNP" H 2950 7317 50  0001 C CNN "D1"
-F 5 "DNP" H 2950 7317 50  0001 C CNN "D1PN"
-F 6 "DNP" H 2900 6900 50  0001 C CNN "MFN"
-F 7 "DNP" H 2900 6900 50  0001 C CNN "MPN"
-	1    2900 6900
-	1    0    0    -1
-$EndComp
-$Comp
-L power:+1V2 #PWR0165
-U 1 1 5CBAB204
-P 3600 6900
-F 0 "#PWR0165" H 3600 6750 50  0001 C CNN
-F 1 "+1V2" H 3615 7073 50  0000 C CNN
-F 2 "" H 3600 6900 50  0001 C CNN
-F 3 "" H 3600 6900 50  0001 C CNN
-	1    3600 6900
 	1    0    0    -1
 $EndComp
@@
 Text GLabel 6650 3400 0    50   Input ~ 0
 BONUS1_EXTCLK
-Text GLabel 3600 4650 2    50   Input ~ 0
+Text GLabel 6650 5000 0    50   Input ~ 0
 BONUS1_RESET
 Text GLabel 6650 3300 0    50   Input ~ 0
 BONUS1_TRIGGER
-Text GLabel 3600 4750 2    50   Input ~ 0
+Text GLabel 6650 5100 0    50   Input ~ 0
 BONUS1_FLASH
 Text GLabel 6650 4600 0    50   Input ~ 0
@@
 Text GLabel 8550 2600 2    50   Input ~ 0
 CAM0_TRIG_1V8
-Text GLabel 6650 5100 0    50   Input ~ 0
+Text GLabel 5400 4650 0    50   Input ~ 0
 BONUS4_SCL0
 Text GLabel 8550 5500 2    50   Input ~ 0
@@
 Text GLabel 6650 5600 0    50   Input ~ 0
 BONUS4_DAT1-
-Text GLabel 6650 5000 0    50   Input ~ 0
+Text GLabel 5400 4550 0    50   Input ~ 0
 BONUS4_EXTCLK
 Text GLabel 8550 4900 2    50   Input ~ 0
@@
 Text GLabel 3600 6150 2    50   Input ~ 0
 AUX3
-Text GLabel 3200 6800 2    50   Input ~ 0
-AUX0
-Text GLabel 2700 6800 0    50   Input ~ 0
-AUX1
-Text GLabel 2700 7000 0    50   Input ~ 0
-AUX3
-Text GLabel 2700 7100 0    50   Input ~ 0
+Text GLabel 3600 5450 2    50   Input ~ 0
 AUX4
-Text GLabel 1750 6050 0    50   Input ~ 0
-AUX4
-Text GLabel 1750 6150 0    50   Input ~ 0
+Text GLabel 3600 5550 2    50   Input ~ 0
 AUX5
-Text GLabel 2700 6900 0    50   Input ~ 0
-AUX2
-Text GLabel 3200 7100 2    50   Input ~ 0
-AUX5
 Wire Wire Line
 	13700 3500 14300 3500
@@
 Wire Wire Line
 	3900 8350 3900 8250
-Wire Wire Line
-	3200 6900 3600 6900
-Wire Wire Line
-	3200 7000 3600 7000
 Connection ~ 14300 3500
 Connection ~ 14300 3000
@@
 	7100 8000 7500 8000
 Connection ~ 7100 8000
+Text GLabel 1750 6050 0    50   Input ~ 0
+LED2
+Text GLabel 1750 6150 0    50   Input ~ 0
+LED3
+Text Notes 1100 6600 0    118  ~ 24
+TODO: assign "AUX" pins to north bonus header
 $EndSCHEMATC

Commit message: working towards front-pack connector as well as backpack connector
Parts:
- added J6: FRONT_PACK, Connector_PinHeader_2.00mm:PinHeader_2x08_P2.00mm_Vertical_SMD, symbol Connector_Generic:Conn_02x08_Odd_Even
Connections:
- net labels added: GPIO18, GPIO19
- net labels removed: AUX0, AUX1, AUX2, AUX3, AUX4, AUX5
- wire segments 206 -> 209
Other:
- note removed: "TODO: assign "AUX" pins to north bonus header"
Changed lines of the file:
@@
 Text GLabel 6650 3300 0    50   Input ~ 0
 BONUS1_TRIGGER
-Text GLabel 6650 5100 0    50   Input ~ 0
-BONUS1_FLASH
 Text GLabel 6650 4600 0    50   Input ~ 0
 BONUS1_SDA1
@@
 Text GLabel 8550 2600 2    50   Input ~ 0
 CAM0_TRIG_1V8
-Text GLabel 5400 4650 0    50   Input ~ 0
+Text GLabel 3600 4750 2    50   Input ~ 0
 BONUS4_SCL0
-Text GLabel 8550 5500 2    50   Input ~ 0
+Text GLabel 3600 5150 2    50   Input ~ 0
 BONUS4_SDA0
-Text GLabel 8550 5900 2    50   Input ~ 0
+Text GLabel 3600 5550 2    50   Input ~ 0
 BONUS4_FLASH
-Text GLabel 8550 6200 2    50   Input ~ 0
+Text GLabel 3600 6150 2    50   Input ~ 0
 BONUS4_TRIGGER
 Text GLabel 8550 2900 2    50   Input ~ 0
@@
 Text GLabel 6650 5600 0    50   Input ~ 0
 BONUS4_DAT1-
-Text GLabel 5400 4550 0    50   Input ~ 0
+Text GLabel 3600 4650 2    50   Input ~ 0
 BONUS4_EXTCLK
 Text GLabel 8550 4900 2    50   Input ~ 0
@@
 Text GLabel 8550 2300 2    50   Input ~ 0
 CAM0_SCL_1V8
-Text GLabel 8550 5800 2    50   Input ~ 0
+Text GLabel 3600 6050 2    50   Input ~ 0
 BONUS4_RESET
 Text GLabel 6650 4500 0    50   Input ~ 0
@@
 Text GLabel 11650 3700 0    50   Input ~ 0
 USB2_D-
-Text GLabel 8550 5600 2    50   Input ~ 0
+Text GLabel 3600 5250 2    50   Input ~ 0
 BONUS4_SCL1
-Text GLabel 6650 5700 0    50   Input ~ 0
-BONUS4_SDA1
 Text GLabel 11650 3300 0    50   Input ~ 0
 GPIO13
@@
 Text Notes 1950 7650 0    118  ~ 24
 boot-select DIP switch
-Text GLabel 3600 5150 2    50   Input ~ 0
-AUX0
-Text GLabel 3600 5250 2    50   Input ~ 0
-AUX1
-Text GLabel 3600 6050 2    50   Input ~ 0
-AUX2
-Text GLabel 3600 6150 2    50   Input ~ 0
-AUX3
-Text GLabel 3600 5450 2    50   Input ~ 0
-AUX4
-Text GLabel 3600 5550 2    50   Input ~ 0
-AUX5
 Wire Wire Line
 	13700 3500 14300 3500
@@
 Text GLabel 1750 6150 0    50   Input ~ 0
 LED3
-Text Notes 1100 6600 0    118  ~ 24
-TODO: assign "AUX" pins to north bonus header
+Text GLabel 3600 5450 2    50   Input ~ 0
+BONUS4_SDA1
+Text GLabel 6650 5100 0    50   Input ~ 0
+BONUS1_FLASH
+$Comp
+L power:GND #PWR0167
+U 1 1 5E9EB5DC
+P 14600 7200
+F 0 "#PWR0167" H 14600 6950 50  0001 C CNN
+F 1 "GND" H 14605 7027 50  0001 C CNN
+F 2 "" H 14600 7200 50  0001 C CNN
+F 3 "" H 14600 7200 50  0001 C CNN
+	1    14600 7200
+	1    0    0    -1
+$EndComp
+Text GLabel 14450 7800 2    50   Input ~ 0
+JTAG_TMS
+Text GLabel 14450 7700 2    50   Input ~ 0
+JTAG_TDI
+Text GLabel 13950 7900 0    50   Input ~ 0
+JTAG_TDO
+Text GLabel 13950 7800 0    50   Input ~ 0
+JTAG_TCK
+Text GLabel 14450 7900 2    50   Input ~ 0
+VCC_JTAG
+Wire Wire Line
+	14600 7200 14450 7200
+$Comp
+L Connector_Generic:Conn_02x08_Odd_Even J6
+U 1 1 5CD032F0
+P 14150 7500
+F 0 "J6" H 14200 8150 50  0000 C CNN
+F 1 "FRONT_PACK" H 14200 8050 50  0000 C CNN
+F 2 "Connector_PinHeader_2.00mm:PinHeader_2x08_P2.00mm_Vertical_SMD" H 14150 7500 50  0001 C CNN
+F 3 "~" H 14150 7500 50  0001 C CNN
+F 4 "Digikey" H 14200 7917 50  0001 C CNN "D1"
+F 5 "S6009-08-ND" H 14200 7917 50  0001 C CNN "D1PN"
+F 6 "NRPN082MAMS-RC" H 14200 7917 50  0001 C CNN "MFN"
+F 7 "Sullins" H 14200 7917 50  0001 C CNN "MPN"
+	1    14150 7500
+	1    0    0    -1
+$EndComp
+Text GLabel 13700 3300 2    50   Input ~ 0
+GPIO18
+Text GLabel 13700 3400 2    50   Input ~ 0
+GPIO19
+Text GLabel 14450 7600 2    50   Input ~ 0
+ROOT_RX
+Text GLabel 14450 7500 2    50   Input ~ 0
+ROOT_TX
+$Comp
+L power:+3.3V #PWR?
+U 1 1 5E3BE12A
+P 13800 7200
+F 0 "#PWR?" H 13800 7050 50  0001 C CNN
+F 1 "+3.3V" H 13815 7373 50  0000 C CNN
+F 2 "" H 13800 7200 50  0001 C CNN
+F 3 "" H 13800 7200 50  0001 C CNN
+	1    13800 7200
+	1    0    0    -1
+$EndComp
+$Comp
+L power:+1V2 #PWR?
+U 1 1 5E3D1866
+P 13550 7300
+F 0 "#PWR?" H 13550 7150 50  0001 C CNN
+F 1 "+1V2" H 13565 7473 50  0000 C CNN
+F 2 "" H 13550 7300 50  0001 C CNN
+F 3 "" H 13550 7300 50  0001 C CNN
+	1    13550 7300
+	1    0    0    -1
+$EndComp
+Wire Wire Line
+	13550 7300 13950 7300
+Wire Wire Line
+	13800 7200 13950 7200
 $EndSCHEMATC

Commit message: finished front-pack connector route
Parts:
- U8: D1PN 296-53432-1-ND -> 296-53472-1-ND; MPN SN74AXC4T245RSVR -> SN74AXC4T245PWR
Connections:
- net labels added: FRONT_AUX0, FRONT_AUX1, FRONT_AUX2, FRONT_AUX3, FRONT_AUX4, FRONT_AUX5
- wire segments 209 -> 210

Commit message: clean up
Parts:
- J6: footprint Connector_PinHeader_2.00mm:PinHeader_2x08_P2.00mm_Vertical_SMD -> Connector_PinHeader_2.00mm:PinHeader_2x08_P2.00mm_Vertical
Other:
- note added: "CS"
- note added: "MISO"
- note added: "MOSI"
- note added: "NRST"
- note added: "SCK"
- note added: "SYNC"

Commit message: add last part number and a few random cleanups
Parts:
- J6: D1PN S6009-08-ND -> S5801-08-ND; MFN NRPN082MAMS-RC -> NRPN082PAEN-RC

Commit message: update part numbers
Parts:
- C14, C15, C53, C69, C70, C71, C72, C73, C74, C85: D1PN 1276-1004-1-ND -> 490-11917-1-ND; MFN Samsung -> Murata; MPN CL05F104ZO5NNNC -> GRM155R61H104KE19D
- M1: D1N (none) -> DNP
- R16, R17, R18, R19, R20, R9: D1PN 311-2.20KLRCT-ND -> P2.20KLCT-ND; MFN Yageo -> Panasonic; MPN RC0402FR-072K2L -> ERJ-2RKF2201X
