File: hardware/ovc4/carrier/power.sch (KiCad schematic (older format))
At the start: 17 parts, among them U1 Jetson_Nano

Commit message: More schematic work
Signed-off-by: Luca Della Vedova <luca@openrobotics.org>
Parts:
- removed SW? (x2): SW_Push, symbol Switch:SW_Push
- added C25, C27: 10u, Capacitor_SMD:C_1206_3216Metric, symbol Device:C_Small
- added C26: todo, Capacitor_SMD:C_0402_1005Metric, symbol Device:C_Small
- added C28: 100n, Capacitor_SMD:C_0402_1005Metric, symbol Device:C_Small
- added C33, C34: 1u, Capacitor_SMD:C_0402_1005Metric, symbol Device:C_Small
- added C63: 560u, Capacitor_SMD:CP_Elec_6.3x7.7, symbol Device:CP1_Small
- added C64: 47u, Capacitor_SMD:C_1206_3216Metric, symbol Device:C_Small
- added J3: Conn_01x02, Connector_PinHeader_2.54mm:PinHeader_1x02_P2.54mm_Vertical, symbol Connector_Generic:Conn_01x02
- added R18: todo, Resistor_SMD:R_0402_1005Metric, symbol Device:R_Small
- added R19, R21, R22, R31: 10k, Resistor_SMD:R_0402_1005Metric, symbol Device:R_Small
- added R20: 56k, Resistor_SMD:R_0402_1005Metric, symbol Device:R_Small
- added R23: 2k4, Resistor_SMD:R_0402_1005Metric, symbol Device:R_Small
- added R24: 22k, Resistor_SMD:R_0402_1005Metric, symbol Device:R_Small
- added R29: 100k, Resistor_SMD:R_0402_1005Metric, symbol Device:R_Small
- added U11: TLV70218_SOT23-5, Package_TO_SOT_SMD:SOT-23-5, symbol Regulator_Linear:TLV70218_SOT23-5
- added U6: 74AHC1G08, Package_TO_SOT_SMD:SOT-353_SC-70-5, symbol 74xGxx:74AHC1G08
- added U7: TPSM53604, DCDC:TI_B3QFN, symbol DCDC_Converters:TPSM53604
- added U8: TPS2121, TI:Texas_VQFN-HR-12_2x2.5_Pitch0.5mm, symbol power_mux:TPS2121
- R25, R27: renamed from R?; value 19k6 -> 21k
- SW1: renamed from SW?; footprint (none) -> Button_Switch_THT:SW_PUSH_6mm
- gave numbers to parts that had none: 11
Connections:
- net +3V3: now also C33.1, R31.1, U11.1 (IN), U11.3 (EN)
- net +5V: now also C63.1, R18.1, R19.1, R29.1, U6.5 (VCC)
- net GND: now also SW1.2, C25.2, C26.2, C27.2, C28.2, C33.2, C34.2, C64.2, J3.2 (Pin_2), R21.2, R23.2, R24.2, U11.2 (GND), U6.3 (GND), U7.10 (NC/GND), U7.11 (NC/GND), U7.12 (AGND), U7.15 (PGND), U7.3 (NC/GND), U8.12 (GND), U8.3 (CP2), U8.4 (OV2), U8.5 (OV1), U8.9 (ST)
- net VBUS: now also U8.2 (IN2)
- net nFORCE_RECOVERY: now also J3.1 (Pin_1)
- net nSHUTDOWN_REQ: now reaches U1.233 (nSHUTDOWN_REQ)
- net POWER_EN: now reaches U1.237 (POWER_EN)
- net POWER_EN: now also U6.4
- net V33_POK: now reaches U9.17 (POK)
- net V33_POK: now also R29.2
- net RST_BUTTON: now reaches SW1.1
- net RST_BUTTON: now also R31.2
- net VCC renamed VREG_5V
- net VREG_5V: now also C64.1, R22.1, U7.7 (VOUT), U7.8 (VOUT)
- new net: C28.1, U8.11 (SS)
- new net: R24.1, U8.10 (ILIM)
- new net: C26.1, R18.2, U6.2
- new net: R22.2, R23.1, U7.9 (FB)
- new net +1V8: C34.1, U11.5 (OUT)
- new net MCU_nPWEN: R19.2, U6.1
- new net PR1: R20.2, R21.1, U8.6 (PR1)
- new net VAUX: R20.1, U8.7 (IN1)
- new net VREG_IN: C25.1, C27.1, U7.1 (VIN), U7.14 (VIN), U7.2 (EN), U8.1 (OUT), U8.8 (OUT)
- no-connect marks 1 -> 5
Other:
- note added: "IN1 is straight from USB bus\nIN2 is regulated from VBUS\nJetson maximum VIN is 5.25V\nNominal OV is 5.5V, high because of low accuracy (+- 5%)\nAutomatic switchover to whichever voltage is higher (with IN2 being preferred)\nCurrent limit at 4.5A"
- note added: "If VAUX is valid (>= 6V) use it in any case\nOtherwise try VBUS\nOV1 / OV2 disabled, regulator can accept 36V, TPS2121 only 21V\nTPS will be damaged before we reach downstream overvoltage"
- note added: "Output capacitance is 1000uF MAX"
- note added: "Set to 5.17V to compensate R losses of series MUX"
- note added: "TODO 20u ceramic is minimum, might increase for safety"
- note added: "TODO battery if we want RTC"
- note added: "TODO sys_reset to MCU\nif we want to reset module"
- note added: "Without MCU only RC delay network\nMCU can turn off / turn on after power on delay"
- note removed: "IN1 is straight from USB bus\nIN2 is regulated from VBUS\nJetson maximum VIN is 5.25V\nNominal OV is 5.21V, get low tol resistors\nAutomatic switchover to whichever voltage is valid (with IN2 being preferred)\nCurrent limit at 4.5A"
- note removed: "TODO bulk cap, 560u on official carrier"
- note removed: "TODO check if we need POK"
- note removed: "TODO check if we need RECOVERY"
- note removed: "TODO series switch for VOUT or ENABLE tied to Jetson nSYS_RESET"
- moved on the sheet: C23, C24, C29, C30, C31, C32, R25, R26, R27, R28, R30, SW1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
