File: hardware/ovc5/carrier/power.kicad_sch (KiCad schematic)
At the start: 27 parts, among them J2 AUX_PWR, U6 TPS2121, U7 TPSM53604RDA, U9 EN5339QI

Commit message: Place and route USB and MIPI lanes
Signed-off-by: Luca Della Vedova <luca@openrobotics.org>
Parts:
- C4: footprint Capacitor_SMD:C_0603_1608Metric -> Capacitor_SMD:C_0402_1005Metric
Changed lines of the file:
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@@
       (effects (font (size 1.27 1.27)) (justify left))
     )
-    (property "Footprint" "Capacitor_SMD:C_0603_1608Metric" (id 2) (at 224.79 40.64 0)
+    (property "Footprint" "Capacitor_SMD:C_0402_1005Metric" (id 2) (at 224.79 40.64 0)
       (effects (font (size 1.27 1.27)) hide)
     )

Commit message: Finished most placing and routing
Signed-off-by: Luca Della Vedova <luca@openrobotics.org>
Parts:
- added C23: 22u, Capacitor_SMD:C_0603_1608Metric, symbol Device:C_Small
Connections:
- net GND: now also C23.2
- net VREG: now reaches C95.1, C96.1, C97.1, R23.1, R25.1, U6.6 (PR1), U6.7 (IN1), U7.7 (VOUT), U7.8 (VOUT)
- net VREG: now also C23.1
Other:
- moved on the sheet: C93, C94, C95, C96, C97, C98, J2, R23, R24, R25, R26, R27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

Commit message: Finish placement and routing
Signed-off-by: Luca Della Vedova <luca@openrobotics.org>
Parts:
- J2: footprint Connector_Molex:Molex_Nano-Fit_105313-xx02_1x02_P2.50mm_Horizontal -> Connector_BarrelJack:BarrelJack_CUI_PJ-102AH_Horizontal; symbol Connector_Generic:Conn_01x02 -> Connector_Generic:Conn_01x03
Connections:
- net GND: now also J2.3 (Pin_3)
Changed lines of the file:
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@@
 (kicad_sch (version 20210126) (generator eeschema)
   (paper "A4")
+  (junction (at 69.85 88.9) (diameter 0.9144) (color 0 0 0 0))
   (junction (at 77.47 83.82) (diameter 0.9144) (color 0 0 0 0))
   (junction (at 77.47 88.9) (diameter 0.9144) (color 0 0 0 0))
@@
     (pin "2")
   )
-  (symbol (lib_id "Connector_Generic:Conn_01x02") (at 64.77 83.82 0) (mirror y) (unit 1)
-    (in_bom yes) (on_board yes)
-    (property "Reference" "J2" (id 0) (at 67.31 77.47 0))
-    (property "Value" "AUX_PWR" (id 1) (at 67.31 80.01 0))
-    (property "Footprint" "Connector_Molex:Molex_Nano-Fit_105313-xx02_1x02_P2.50mm_Horizontal" (id 2) (at 64.77 83.82 0)
-      (effects (font (size 1.27 1.27)) hide)
-    )
-    (property "Datasheet" "~" (id 3) (at 64.77 83.82 0)
-      (effects (font (size 1.27 1.27)) hide)
-    )
-    (pin "1")
-    (pin "2")
+  (symbol (lib_id "Connector_Generic:Conn_01x03") (at 64.77 86.36 0) (mirror y) (unit 1)
+    (in_bom yes) (on_board yes)
+    (property "Reference" "J2" (id 0) (at 67.31 80.01 0))
+    (property "Value" "AUX_PWR" (id 1) (at 67.31 82.55 0))
+    (property "Footprint" "Connector_BarrelJack:BarrelJack_CUI_PJ-102AH_Horizontal" (id 2) (at 64.77 86.36 0)
+      (effects (font (size 1.27 1.27)) hide)
+    )
+    (property "Datasheet" "~" (id 3) (at 64.77 86.36 0)
+      (effects (font (size 1.27 1.27)) hide)
+    )
+    (pin "1")
+    (pin "2")
+    (pin "3")
   )
   (symbol (lib_id "power_mux:TPS2121") (at 194.31 90.17 0) (unit 1)

Commit message: Add parts for BOM
Signed-off-by: Luca Della Vedova <luca@openrobotics.org>
Parts:
- C2: D1N (none) -> Digikey; D1PN (none) -> 1276-1076-1-ND; MFN (none) -> Samsung; MPN (none) -> CL05A105KP5NNNC
- C23, C3, C5, C6, C7, C95, C96, C97: D1N (none) -> Digikey; D1PN (none) -> 1276-6504-1-ND; MFN (none) -> Samsung; MPN (none) -> CL10A226MPCNUBE
- C4: D1N (none) -> Digikey; D1PN (none) -> 587-1947-1-ND; MFN (none) -> Taiyo Yuden; MPN (none) -> UMK105CG100DV-F
- C8, C98: D1N (none) -> Digikey; D1PN (none) -> 1276-1043-1-ND; MFN (none) -> Samsung; MPN (none) -> CL05A104KA5NNNC
- C93, C94: D1N (none) -> Digikey; D1PN (none) -> 1276-2876-1-ND; MFN (none) -> Samsung; MPN (none) -> CL31A106KBHNNNE
- J2: D1N (none) -> Digikey; D1PN (none) -> CP-102AH-ND; MFN (none) -> CUI Devices; MPN (none) -> PJ-102AH
- R2, R3: D1N (none) -> Digikey; D1PN (none) -> 2019-RK73H1ETTP3483FCT-ND; MFN (none) -> KOA Speer; MPN (none) -> RK73H1ETTP3483F
- R23, R26, R28: D1N (none) -> Digikey; D1PN (none) -> YAG3436CT-ND; MFN (none) -> Yageo; MPN (none) -> AC0402FR-0710KL
- R24: D1N (none) -> Digikey; D1PN (none) -> P2.43KDCCT-ND; MFN (none) -> Panasonic; MPN (none) -> ERA-2AEB2431X
- R25, R27: D1N (none) -> Digikey; D1PN (none) -> 311-47.0KLRCT-ND; MFN (none) -> Yageo; MPN (none) -> RC0402FR-0747KL
- R29: value 22k -> 20k; D1N (none) -> Digikey; D1PN (none) -> 311-20.0KLRCT-ND; MFN (none) -> Yageo; MPN (none) -> RC0402FR-0720KL
- R4: D1N (none) -> Digikey; D1PN (none) -> YAG3515CT-ND; MFN (none) -> Yageo; MPN (none) -> YAG3515CT-ND
- U6: D1N (none) -> Digikey; D1PN (none) -> 296-53410-1-ND; MFN (none) -> TI; MPN (none) -> TPS2121RUXR
- U7: D1N (none) -> Digikey; D1PN (none) -> 296-TPSM53604RDARCT-ND; MFN (none) -> TI; MPN (none) -> TPSM53604RDAR
- U9: D1N (none) -> Digikey; D1PN (none) -> 544-2854-1-ND; MFN (none) -> Intel; MPN (none) -> EN5339QI

Commit message: Routing and FPGA pin assignment optimizations
Also fixed some pins that were NC by accident

Signed-off-by: Luca Della Vedova <luca@openrobotics.org>
Parts:
- R4: value 100k -> 47k; D1PN YAG3515CT-ND -> 311-47.0KLRCT-ND; MPN YAG3515CT-ND -> RC0402FR-0747KL
Changed lines of the file:
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@@
       (effects (font (size 1.27 1.27)) (justify left))
     )
-    (property "Value" "100k" (id 1) (at 185.42 35.56 0)
+    (property "Value" "47k" (id 1) (at 185.42 35.56 0)
       (effects (font (size 1.27 1.27)) (justify left))
     )
@@
       (effects (font (size 1.27 1.27)) hide)
     )
-    (property "D1PN" "YAG3515CT-ND" (id 5) (at 182.88 34.29 0)
+    (property "D1PN" "311-47.0KLRCT-ND" (id 5) (at 182.88 34.29 0)
       (effects (font (size 1.27 1.27)) hide)
     )
@@
       (effects (font (size 1.27 1.27)) hide)
     )
-    (property "MPN" "YAG3515CT-ND" (id 7) (at 182.88 34.29 0)
+    (property "MPN" "RC0402FR-0747KL" (id 7) (at 182.88 34.29 0)
       (effects (font (size 1.27 1.27)) hide)
     )

Commit message: Address feedback
Fix oscillator circuit
Fix skew in MIPI lane

Signed-off-by: Luca Della Vedova <luca@openrobotics.org>
Parts:
- R24: value 2k43 -> 2k4; D1PN P2.43KDCCT-ND -> P2.4KDECT-ND; MPN ERA-2AEB2431X -> ERA-2AED242X
Other:
- note added: "Set to 5.17V for MUX series loss"
- note removed: "Set to 5.11V for MUX series loss"
Changed lines of the file:
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@@
     (stroke (width 0) (type solid) (color 0 0 0 0))
   )
-  (text "Set to 5.11V for MUX series loss" (at 128.27 73.66 180)
+  (text "Set to 5.17V for MUX series loss" (at 128.27 73.66 180)
     (effects (font (size 1.27 1.27)) (justify right bottom))
   )
@@
       (effects (font (size 1.27 1.27)) (justify left))
     )
-    (property "Value" "2k43" (id 1) (at 129.54 96.52 0)
+    (property "Value" "2k4" (id 1) (at 129.54 96.52 0)
       (effects (font (size 1.27 1.27)) (justify left))
     )
@@
       (effects (font (size 1.27 1.27)) hide)
     )
-    (property "D1PN" "P2.43KDCCT-ND" (id 5) (at 127 95.25 0)
+    (property "D1PN" "P2.4KDECT-ND" (id 5) (at 127 95.25 0)
       (effects (font (size 1.27 1.27)) hide)
     )
@@
       (effects (font (size 1.27 1.27)) hide)
     )
-    (property "MPN" "ERA-2AEB2431X" (id 7) (at 127 95.25 0)
-      (effects (font (size 1.27 1.27)) hide)
-    )
+    (property "MPN" "ERA-2AED242X" (id 7) (at 127 95.25 0)
+      (effects (font (size 1.27 1.27)) hide)
+    )
