File: hardware/ovc5/carrier/usb.kicad_sch (KiCad schematic)
At the start: 3 parts, among them J1 USB_C_Receptacle, U2 CYUSB43x7, U5 USB3_A_Dual_Stacked

Commit message: Finish main schematics, start placing
Signed-off-by: Luca Della Vedova <luca@openrobotics.org>
Parts:
- added C1, C10, C11, C12, C13, C14, C15, C16, C17, C18, C19, C20, C21, C22, C23, C24, C30, C32, C36, C37, C38, C39, C40, C41, C42, C43, C44, C45, C48, C49, C50, C52, C53, C54, C56, C57, C59, C60, C61, C65, C66, C67, C68, C70, C74, C75, C76, C77, C79, C80, C81, C82: 100n, Capacitor_SMD:C_0402_1005Metric, symbol Device:C_Small
- added C25, C34, C47: 10u, Capacitor_SMD:C_0402_1005Metric, symbol Device:C_Small
- added C26, C27, C28, C46, C51: 10n, Capacitor_SMD:C_0402_1005Metric, symbol Device:C_Small
- added C29, C31, C62: 4u7, Capacitor_SMD:C_0402_1005Metric, symbol Device:C_Small
- added C33, C35, C55, C58, C9: 1u, Capacitor_SMD:C_0402_1005Metric, symbol Device:C_Small
- added C63, C64: 12pF, Capacitor_SMD:C_0402_1005Metric, symbol Device:C_Small
- added C69, C71: 100u, Capacitor_SMD:C_1206_3216Metric, symbol Device:C_Small
- added C72, C73: 2n2, Capacitor_SMD:C_0402_1005Metric, symbol Device:C_Small
- added R1: 47k, Resistor_SMD:R_0402_1005Metric, symbol Device:R_Small
- added R10, R5: 20k, Resistor_SMD:R_0402_1005Metric, symbol Device:R_Small
- added R11, R12, R17, R18, R8, R9: 100k, Resistor_SMD:R_0402_1005Metric, symbol Device:R_Small
- added R13, R15, R44, R6, R7: 10k, Resistor_SMD:R_0402_1005Metric, symbol Device:R_Small
- added R14, R16: 1k, Resistor_SMD:R_0402_1005Metric, symbol Device:R_Small
- added R19, R20: 5k1, Resistor_SMD:R_0402_1005Metric, symbol Device:R_Small
- added R42, R43: 2k4, Resistor_SMD:R_0402_1005Metric, symbol Device:R_Small
- added U10: S25FL064, Package_SON:WSON-8-1EP_6x5mm_P1.27mm_EP3.4x4mm, symbol memory_eeprom:S25FL064
- added U8: TPS2561, Package_SON:VSON-10-1EP_3x3mm_P0.5mm_EP1.65x2.4mm_ThermalVias, symbol Interface_USB:TPS2561
- added Y1: 25MHz, Crystal:Crystal_SMD_2016-4Pin_2.0x1.6mm, symbol Device:Crystal_Small
Connections:
- net USB_UART_D-: now reaches U2.A12 (D_P6_N)
- net USB_UART_D+: now reaches U2.A13 (D_P6_P)
- net FPGA_USB0_D-: now reaches U2.B1 (D_P1_N)
- net FPGA_USB1_D-: now reaches U2.B13 (D_P2_N)
- net FPGA_USB1_D+: now reaches U2.B14 (D_P2_P)
- net FPGA_USB0_D+: now reaches U2.B2 (D_P1_P)
- net USB_DS_CC2: now reaches U2.B3 (CC2_P0)
- net USB_DS_CC2: now also J1.B5 (CC2)
- net VBUS_MON_P1: now reaches U2.B5 (VBUS_MON_P1)
- net VBUS_MON_P1: now also C67.1, R15.1, R16.2
- net FPGA_USB0_TX+: now reaches U2.C1 (TX1_P1_P)
- net FPGA_USB0_TX-: now reaches U2.C2 (TX1_P1_N)
- net +3V3: now reaches U2.C6 (OCP_DET_P1)
- net +3V3: now also U2.A5 (VDDD_PD), U2.C12 (VDDIO), U2.C3 (VDDIO), U2.C9 (VDDD_DMC), U2.E8 (AVDD33), U2.F10 (OVCUR_P2), U2.G12 (V3P3), U2.G3 (V3P3), U2.G5 (OCP_DET_P0), U2.H10 (OVCUR_P6), U2.J12 (VDDIO), U2.K11 (PSELF), U2.K6 (OVCUR_P1), U2.L10 (VDDIO), U2.L12 (V3P3), U2.L3 (V3P3), U2.M11 (OVCUR_P7), U2.M3 (V3P3), U2.N12 (OVCUR_P3), U2.P10 (V3P3_REG), C41.1, C42.1, C43.1, C44.1, C45.1, C46.1, C47.1, C48.1, C49.1, C50.1, C51.1, C52.1, C53.1, C54.1, C55.1, C56.1, C58.1, C60.1, C65.1, R11.1, R12.1, R42.1, R43.1, R44.2, R5.1, R6.1, R7.1, R8.1, R9.1, U10.8 (VCC)
- net FPGA_USB0_RX+: now reaches U2.D1 (RX1_P1_P)
- net FPGA_USB0_RX-: now reaches U2.D2 (RX1_P1_N)
- net USB_DS_CC1: now reaches U2.D3 (CC1_P0)
- net USB_DS_CC1: now also J1.A5 (CC1)
- net VBUS_MON_P0: now reaches U2.D4 (VBUS_MON_P0)
- net VBUS_MON_P0: now also C66.1, R13.1, R14.2
- net at U2.D5 (VSEL_GPIO1): now also U2.F5 (VSEL_GPIO2), R44.1
- net USB_US0_CC1: now reaches U2.D8 (CC1_P1)
- net USB_US0_CC1: now also R19.1
- net FPGA_USB1_RX-: now reaches U2.E13 (RX1_P2_N)
- net FPGA_USB1_RX+: now reaches U2.E14 (RX1_P2_P)
- net FPGA_USB1_TX-: now reaches U2.F13 (TX1_P2_N)
- net FPGA_USB1_TX+: now reaches U2.F14 (TX1_P2_P)
- net USB_H1_TX_P: now reaches U2.G1 (TX_P5_P)
- net USB_H1_TX_P: now also C82.2
- net USB_H0_RX_N: now reaches U2.G13 (RX_P4_N)
- net USB_H0_RX_N: now also U5.5 (SSRX0-)
- net USB_H0_RX_P: now reaches U2.G14 (RX_P4_P)
- net USB_H0_RX_P: now also U5.6 (SSRX0+)
- net USB_H1_TX_N: now reaches U2.G2 (TX_P5_N)
- net USB_H1_TX_N: now also C80.2
- net USB_H1_RX_P: now reaches U2.H1 (RX_P5_P)
- net USB_H1_RX_P: now also U5.15 (SSRX1+)
- net USB_H0_TX_N: now reaches U2.H13 (TX_P4_N)
- net USB_H0_TX_N: now also C79.2
- net USB_H0_TX_P: now reaches U2.H14 (TX_P4_P)
- net USB_H0_TX_P: now also C81.2
- net USB_H1_RX_N: now reaches U2.H2 (RX_P5_N)
- net USB_H1_RX_N: now also U5.14 (SSRX1-)
- net USB_H1_D_N: now reaches U2.J1 (D_P5_P)
- net USB_H1_D_N: now also U5.11 (D1-)
- net USB_H0_D_N: now reaches U2.J13 (D_P4_N)
- net USB_H0_D_N: now also U5.2 (D0-)
- net USB_H0_D_P: now reaches U2.J14 (D_P4_P)
- net USB_H0_D_P: now also U5.3 (D0+)
- net USB_H1_D_P: now reaches U2.J2 (D_P5_N)
- net USB_H1_D_P: now also U5.12 (D1+)
- net USB_DS_D_N: now reaches U2.K1 (D_P0_N)
- net USB_DS_D_N: now also J1.A7 (D-), J1.B7 (D-)
- net USB_DS_D_P: now reaches U2.K2 (D_P0_P)
- net USB_DS_D_P: now also J1.A6 (D+), J1.B6 (D+)
- net USB_US1_CC1: now reaches U2.K9 (CC1_P2)
- net USB_US1_CC1: now also R20.1
- net USB_DS_TX1_P: now reaches U2.L1 (TX1_P0_P)
- net USB_DS_TX1_P: now also C76.2
- net USB_DS_TX1_N: now reaches U2.L2 (TX1_P0_N)
- net USB_DS_TX1_N: now also C74.2
- net nOVC1: now reaches U2.L5 (OVCUR_P5)
- net nOVC1: now also R9.2, U8.6 (~FAULT2)
- net USBEN1: now reaches U2.L6 (PWREN_P5)
- net USBEN1: now also R11.2, U8.5 (EN2)
- net nOVC0: now reaches U2.L7 (OVCUR_P4)
- net nOVC0: now also R8.2, U8.10 (~FAULT1)
- net USB_DS_RX1_P: now reaches U2.M1 (RX1_P0_P)
- net USB_DS_RX1_P: now also J1.B11 (RX1+)
- net USB_DS_RX1_N: now reaches U2.M2 (RX1_P0_N)
- net USB_DS_RX1_N: now also J1.B10 (RX1-)
- net +5V: now reaches U2.M7 (VBUS)
- net +5V: now also U2.C4 (V5P0_P0), U2.D7 (V5P0_P1), U2.E7 (V5P0), C1.1, C34.1, C36.1, R15.2, U8.2 (IN), U8.3 (IN)
- net USB_DS_RX2_N: now reaches U2.N1 (RX2_P0_N)
- net USB_DS_RX2_N: now also J1.A10 (RX2-)
- net USB_DS_RX2_P: now reaches U2.N2 (RX2_P0_P)
- net USB_DS_RX2_P: now also J1.A11 (RX2+)
- net USBEN0: now reaches U2.N3 (PWREN_P4)
- net USBEN0: now also R12.2, U8.4 (EN1)
- net USB_DS_TX2_N: now reaches U2.P2 (TX2_P0_N)
- net USB_DS_TX2_N: now also C75.2
- net USB_DS_TX2_P: now reaches U2.P3 (TX2_P0_P)
- net USB_DS_TX2_P: now also C77.2
- net VBUS_0: now reaches U5.1 (VBUS0)
- net VBUS_0: now also C68.1, C69.1, U8.9 (OUT1)
- net VBUS_1: now reaches U5.10 (VBUS1)
- net VBUS_1: now also C70.1, C71.1, U8.8 (OUT2)
- net GND: now reaches U5.13 (GND1)
- net GND: now also J1.A1 (GND), J1.A12 (GND), J1.B1 (GND), J1.B12 (GND), U2.E10 (PGANG), U2.F6 (GND), U2.F7 (GND), U2.F8 (GND), U2.F9 (GND), U2.G6 (GND), U2.G7 (GND), U2.G8 (GND), U2.G9 (GND), U2.H6 (GND), U2.H7 (GND), U2.H8 (GND), U2.H9 (GND), U2.J7 (GND), U2.J8 (GND), U2.J9 (GND), U2.N10 (RES/GND), U5.16 (GND1), U5.4 (GND0), U5.7 (GND0), C1.2, C10.2, C11.2, C12.2, C13.2, C14.2, C15.2, C16.2, C17.2, C18.2, C19.2, C20.2, C21.2, C22.2, C23.2, C24.2, C25.2, C26.2, C27.2, C28.2, C29.2, C30.2, C31.2, C32.2, C33.2, C34.2, C35.2, C36.2, C37.2, C38.2, C39.2, C40.2, C41.2, C42.2, C43.2, C44.2, C45.2, C46.2, C47.2, C48.2, C49.2, C50.2, C51.2, C52.2, C53.2, C54.2, C55.2, C56.2, C57.2, C58.2, C59.2, C60.2, C61.2, C62.2, C63.1, C64.2, C65.2, C68.2, C69.2, C70.2, C71.2, C72.2, C73.2, C9.2, R1.2, R10.2, R17.2, R18.2, R19.2, R20.2, U10.4 (VSS), U8.1 (GND), U8.11 (PAD)
- net at U5.17 (SSTX1-): now also C80.1
- net at U5.18 (SSTX1+): now also C82.1
- net at U5.8 (SSTX0-): now also C79.1
- net at U5.9 (SSTX0+): now also C81.1
- net at U5.S (Shield): now also C72.1, R17.1
- net at U2.B6 (VCCD_PD): now also C35.1
- net at U2.D9 (VCCD_DMC): now also C33.1
- net VDD10: now reaches U2.F11 (DVDD10)
- net VDD10: now also U2.F4 (DVDD10), U2.J11 (DVDD10), U2.J4 (DVDD10), C57.1, C59.1, C61.1, C62.1
- net 1V0_PHY: now reaches U2.G11 (V1P0_P6)
- net 1V0_PHY: now also U2.G4 (V1P0_P7), U2.H11 (V1P0_P2), U2.H12 (V1P0_P2), U2.H3 (V1P0_P1), U2.J3 (V1P0_P1), U2.K12 (V1P0_P4), U2.K3 (V1P0_P5), U2.K8 (AVDD10), U2.L11 (V1P0_P3), U2.L4 (V1P0_P0), U2.M12 (V1P0_P3), U2.M4 (V1P0_P0), U2.N8 (V1P0_PHY), U2.N9 (V1P0_PHY), U2.P8 (V1P0_PHY), U2.P9 (V1P0_PHY), C12.1, C13.1, C14.1, C15.1, C16.1, C17.1, C18.1, C19.1, C20.1, C21.1, C22.1, C23.1, C24.1, C25.1, C26.1, C27.1, C28.1
- net V1P0_MEM_B: now reaches U2.N4 (V1P0_MEM_B)
- net V1P0_MEM_B: now also C31.1, C32.1
- net V1P0_MEM_A: now reaches U2.N5 (V1P0_MEM_A)
- net V1P0_MEM_A: now also C29.1, C30.1
- net +1V2: now reaches U2.N6 (V1P2)
- net +1V2: now also U2.P4 (V1P2), U2.P5 (V1P2), U2.P6 (V1P2), C37.1, C38.1, C39.1, C40.1
- net USB_SPI_DO: now reaches U2.A10 (SPI_MISO_DMC)
- net USB_SPI_DO: now also U2.J5 (SPI_MISO_HUB), U10.2 (SO)
- net USB_SP_nWP: now reaches U2.A11 (DMC_P24)
- net USB_SP_nWP: now also U10.3 (nWP)
- net at U2.A6 (XIN): now also C63.2, Y1.2
- net at U2.A7 (XOUT): now also C64.1, Y1.1
- net USB_SPI_CS: now reaches U2.B10 (SPI_SS_DMC)
- net USB_SPI_CS: now also U2.M6 (SPI_SS_HUB), U10.1 (nCS)
- net XRES_DMC: now reaches U2.C11 (XRES_DMC)
- net XRES_DMC: now also C10.1, R6.2
- net USB_I2C_SDA: now reaches U2.D11 (I2C_SDA1)
- net USB_I2C_SDA: now also U2.G10 (I2C_SDA_HUB), R43.2
- net USB_SPI_CLK: now reaches U2.D12 (SPI_CLK_DMC)
- net USB_SPI_CLK: now also U2.K7 (SPI_CLK_HUB), U10.6 (SCK)
- net USB_I2C_SCL: now reaches U2.E11 (I2C_SCL1)
- net USB_I2C_SCL: now also U2.M5 (I2C_SCL_HUB), R42.2
- net USB_SPI_DI: now reaches U2.F12 (SPI_MOSI_DMC)
- net USB_SPI_DI: now also U2.H5 (SPI_MOSI_HUB), U10.5 (SI)
- net XRES_PD: now reaches U2.K4 (XRES_PD)
- net XRES_PD: now also C11.1, R7.2
- net at U2.M10 (RTERM): now also R10.1
- net RESET_HUB: now reaches U2.M8 (RESET_HUB)
- net RESET_HUB: now also C9.1, R5.2
- net at J1.A2 (TX1+): now also C76.1
- net at J1.A3 (TX1-): now also C74.1
- net VBUS: now reaches J1.A4 (VBUS), J1.A9 (VBUS), J1.B4 (VBUS), J1.B9 (VBUS)
- net VBUS: now also R13.2
- net at J1.B2 (TX2+): now also C77.1
- net at J1.B3 (TX2-): now also C75.1
- net at J1.S1 (SHIELD): now also C73.1, R18.1
- new net: R1.1, U8.7 (ILM)
- new net: C67.2, R16.1
- new net: C66.2, R14.1
- no-connect marks 0 -> 54
Other:
- note added: "1.2A limit"
- note added: "CC2 open, CC1 pull-down port unflipped"
- note added: "DS1 always connected"
- note added: "Discharge unimplemented"
- note added: "TODO FTDI UART-Serial in P6, check P7"
- note added: "TODO P25 LED?"
- note added: "TODO check VBUS capacitance and USB spec"
- note added: "TODO check VBUS port"
- note added: "V3P3"
- note added: "VDDIO / V3P3_REG"
- note added: "VDD_DMC"
- note added: "VDD_PD"
- moved on the sheet: J1, U2A, U2B, U2C, U5

Commit message: Place and route USB and MIPI lanes
Signed-off-by: Luca Della Vedova <luca@openrobotics.org>
Parts:
- removed C23: 100n, Capacitor_SMD:C_0402_1005Metric, symbol Device:C_Small
- added D3, D4, D5: D_TVS_Dual_AAC, USB:TPD2EUSB30x, symbol Device:D_TVS_Dual_AAC
Connections:
- net +3V3: now also U2.L7 (OVCUR_P4); no longer U2.C6 (OCP_DET_P1), U2.G5 (OCP_DET_P0), U2.K6 (OVCUR_P1)
- net +5V: no longer R15.2
- net FPGA_USB0_D+: now also U2.J14 (D_P4_P); no longer U2.B2 (D_P1_P)
- net FPGA_USB0_D-: now also U2.J13 (D_P4_N); no longer U2.B1 (D_P1_N)
- net FPGA_USB0_RX+: now also U2.G13 (RX_P4_N); no longer U2.D1 (RX1_P1_P)
- net FPGA_USB0_RX-: now also U2.G14 (RX_P4_P); no longer U2.D2 (RX1_P1_N)
- net FPGA_USB0_TX+: now also U2.H14 (TX_P4_P); no longer U2.C1 (TX1_P1_P)
- net FPGA_USB0_TX-: now also U2.H13 (TX_P4_N); no longer U2.C2 (TX1_P1_N)
- net FPGA_USB1_D+: now also U2.K14 (D_P3_P); no longer U2.B14 (D_P2_P)
- net FPGA_USB1_D-: now also U2.K13 (D_P3_N); no longer U2.B13 (D_P2_N)
- net FPGA_USB1_RX+: now also U2.N13 (RX1_P3_P); no longer U2.E14 (RX1_P2_P)
- net FPGA_USB1_RX-: now also U2.N14 (RX1_P3_N); no longer U2.E13 (RX1_P2_N)
- net FPGA_USB1_TX+: now also U2.P13 (TX1_P3_N); no longer U2.F14 (TX1_P2_P)
- net FPGA_USB1_TX-: now also U2.P12 (TX1_P3_P); no longer U2.F13 (TX1_P2_N)
- net GND: now also D3.3 (common), D4.3 (common), D5.3 (common)
- net USBEN0: now also U2.J6 (PWREN_P1); no longer U2.N3 (PWREN_P4)
- net USB_DS_D_N: now also D3.2 (A2)
- net USB_DS_D_P: now also D3.1 (A1)
- net USB_DS_TX1_N: now also C76.2; no longer C74.2
- net USB_DS_TX1_P: now also C74.2; no longer C76.2
- net USB_DS_TX2_N: now also C77.2; no longer C75.2
- net USB_DS_TX2_P: now also C75.2; no longer C77.2
- net USB_H0_D_N: now also U2.B1 (D_P1_N), U5.11 (D1-), D4.2 (A2); no longer U2.J13 (D_P4_N), U5.2 (D0-)
- net USB_H0_D_P: now also U2.B2 (D_P1_P), U5.12 (D1+), D4.1 (A1); no longer U2.J14 (D_P4_P), U5.3 (D0+)
- net USB_H0_RX_N: now also U2.D2 (RX1_P1_N), U5.14 (SSRX1-); no longer U2.G13 (RX_P4_N), U5.5 (SSRX0-)
- net USB_H0_RX_P: now also U2.D1 (RX1_P1_P), U5.15 (SSRX1+); no longer U2.G14 (RX_P4_P), U5.6 (SSRX0+)
- net USB_H0_TX_N: now also U2.C2 (TX1_P1_N); no longer U2.H13 (TX_P4_N)
- net USB_H0_TX_P: now also U2.C1 (TX1_P1_P); no longer U2.H14 (TX_P4_P)
- net USB_H1_D_N: now also U5.2 (D0-), D5.2 (A2); no longer U5.11 (D1-)
- net USB_H1_D_P: now also U5.3 (D0+), D5.1 (A1); no longer U5.12 (D1+)
- net USB_H1_RX_N: now also U5.5 (SSRX0-); no longer U5.14 (SSRX1-)
- net USB_H1_RX_P: now also U5.6 (SSRX0+); no longer U5.15 (SSRX1+)
- net VBUS_0: now also R15.2, U5.10 (VBUS1); no longer U5.1 (VBUS0)
- net VBUS_1: now also U5.1 (VBUS0); no longer U5.10 (VBUS1)
- net nOVC0: now also U2.K6 (OVCUR_P1); no longer U2.L7 (OVCUR_P4)
- net USB_DS_TX1_CONN_N: now reaches C76.1, J1.A2 (TX1+)
- net at R44.1, U2.D5 (VSEL_GPIO1), U2.F5 (VSEL_GPIO2): now also U2.C6 (OCP_DET_P1), U2.G5 (OCP_DET_P0)
- net USB_DS_TX2_CONN_N: now reaches C77.1, J1.B2 (TX2+)
- net USB_DS_TX2_CONN_P: now reaches C75.1, J1.B3 (TX2-)
- net USB_DS_TX1_CONN_P: now reaches C74.1, J1.A3 (TX1-)
- net USB_H0_TX_CONN_N: now reaches C79.1
- net USB_H0_TX_CONN_N: now also U5.17 (SSTX1-); no longer U5.8 (SSTX0-)
- net USB_H1_TX_CONN_N: now reaches C80.1
- net USB_H1_TX_CONN_N: now also U5.8 (SSTX0-); no longer U5.17 (SSTX1-)
- net USB_H0_TX_CONN_P: now reaches U5.18 (SSTX1+)
- net USB_H0_TX_CONN_P: now also C81.1; no longer C82.1
- net USB_H1_TX_CONN_P: now reaches U5.9 (SSTX0+)
- net USB_H1_TX_CONN_P: now also C82.1; no longer C81.1
- net at C63.2, U2.A6 (XIN): now also Y1.1; no longer Y1.2
- net at C64.1, U2.A7 (XOUT): now also Y1.2; no longer Y1.1
Other:
- note added: "NOTE bypass capacitors for unused port removed (P7)"
- note added: "Pair swapping OK"
- note added: "Polarity swap OK"
- moved on the sheet: C1, C65, C68, C69, C70, C71, C72, C73, C74, C75, C76, C77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

Commit message: Finished most placing and routing
Signed-off-by: Luca Della Vedova <luca@openrobotics.org>
Parts:
- removed C72, C73: 2n2, Capacitor_SMD:C_0402_1005Metric, symbol Device:C_Small
- removed R17, R18: 100k, Resistor_SMD:R_0402_1005Metric, symbol Device:R_Small
Connections:
- net GND: now also J1.S1 (SHIELD), U5.S (Shield)
Changed lines of the file:
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@@
   (junction (at 170.18 149.86) (diameter 0.9144) (color 0 0 0 0))
   (junction (at 170.18 152.4) (diameter 0.9144) (color 0 0 0 0))
-  (junction (at 170.18 260.35) (diameter 0.9144) (color 0 0 0 0))
-  (junction (at 170.18 265.43) (diameter 0.9144) (color 0 0 0 0))
   (junction (at 173.99 0) (diameter 0.9144) (color 0 0 0 0))
   (junction (at 177.8 -5.08) (diameter 0.9144) (color 0 0 0 0))
   (junction (at 177.8 0) (diameter 0.9144) (color 0 0 0 0))
-  (junction (at 177.8 265.43) (diameter 0.9144) (color 0 0 0 0))
+  (junction (at 177.8 260.35) (diameter 0.9144) (color 0 0 0 0))
   (junction (at 179.07 -21.59) (diameter 0.9144) (color 0 0 0 0))
   (junction (at 179.07 -16.51) (diameter 0.9144) (color 0 0 0 0))
@@
   (junction (at 316.23 241.3) (diameter 0.9144) (color 0 0 0 0))
   (junction (at 318.77 241.3) (diameter 0.9144) (color 0 0 0 0))
-  (junction (at 321.31 236.22) (diameter 0.9144) (color 0 0 0 0))
-  (junction (at 321.31 241.3) (diameter 0.9144) (color 0 0 0 0))
   (junction (at 334.01 147.32) (diameter 0.9144) (color 0 0 0 0))
   (junction (at 353.06 147.32) (diameter 0.9144) (color 0 0 0 0))
@@
     (stroke (width 0) (type solid) (color 0 0 0 0))
   )
-  (wire (pts (xy 162.56 260.35) (xy 170.18 260.35))
-    (stroke (width 0) (type solid) (color 0 0 0 0))
-  )
-  (wire (pts (xy 162.56 265.43) (xy 170.18 265.43))
-    (stroke (width 0) (type solid) (color 0 0 0 0))
-  )
   (wire (pts (xy 163.83 50.8) (xy 170.18 50.8))
     (stroke (width 0) (type solid) (color 0 0 0 0))
@@
     (stroke (width 0) (type solid) (color 0 0 0 0))
   )
+  (wire (pts (xy 170.18 260.35) (xy 177.8 260.35))
+    (stroke (width 0) (type solid) (color 0 0 0 0))
+  )
   (wire (pts (xy 173.99 0) (xy 173.99 2.54))
     (stroke (width 0) (type solid) (color 0 0 0 0))
@@
     (stroke (width 0) (type solid) (color 0 0 0 0))
   )
-  (wire (pts (xy 177.8 259.08) (xy 177.8 265.43))
-    (stroke (width 0) (type solid) (color 0 0 0 0))
-  )
-  (wire (pts (xy 177.8 265.43) (xy 170.18 265.43))
+  (wire (pts (xy 177.8 259.08) (xy 177.8 260.35))
     (stroke (width 0) (type solid) (color 0 0 0 0))
   )
-  (wire (pts (xy 177.8 265.43) (xy 177.8 266.7))
+  (wire (pts (xy 177.8 260.35) (xy 177.8 266.7))
     (stroke (width 0) (type solid) (color 0 0 0 0))
   )
@@
     (stroke (width 0) (type solid) (color 0 0 0 0))
   )
-  (wire (pts (xy 318.77 241.3) (xy 321.31 241.3))
+  (wire (pts (xy 321.31 233.68) (xy 321.31 241.3))
     (stroke (width 0) (type solid) (color 0 0 0 0))
   )
-  (wire (pts (xy 321.31 233.68) (xy 321.31 236.22))
-    (stroke (width 0) (type solid) (color 0 0 0 0))
-  )
-  (wire (pts (xy 321.31 236.22) (xy 328.93 236.22))
-    (stroke (width 0) (type solid) (color 0 0 0 0))
-  )
-  (wire (pts (xy 321.31 241.3) (xy 328.93 241.3))
+  (wire (pts (xy 321.31 241.3) (xy 318.77 241.3))
     (stroke (width 0) (type solid) (color 0 0 0 0))
   )
@@
     (pin "2")
   )
-  (symbol (lib_id "Device:R_Small") (at 162.56 262.89 0) (unit 1)
-    (in_bom yes) (on_board yes)
-    (property "Reference" "R18" (id 0) (at 165.1 259.08 0)
-      (effects (font (size 1.27 1.27)) (justify left))
-    )
-    (property "Value" "100k" (id 1) (at 163.83 261.62 0)
-      (effects (font (size 1.27 1.27)) (justify left))
-    )
-    (property "Footprint" "Resistor_SMD:R_0402_1005Metric" (id 2) (at 162.56 262.89 0)
-      (effects (font (size 1.27 1.27)) hide)
-    )
-    (property "Datasheet" "~" (id 3) (at 162.56 262.89 0)
-      (effects (font (size 1.27 1.27)) hide)
-    )
-    (pin "1")
-    (pin "2")
-  )
   (symbol (lib_id "Device:R_Small") (at 250.19 151.13 0) (unit 1)
     (in_bom yes) (on_board yes)
@@
     (pin "2")
   )
-  (symbol (lib_id "Device:R_Small") (at 321.31 238.76 0) (unit 1)
-    (in_bom yes) (on_board yes)
-    (property "Reference" "R17" (id 0) (at 323.85 234.95 0)
-      (effects (font (size 1.27 1.27)) (justify left))
-    )
-    (property "Value" "100k" (id 1) (at 322.58 237.49 0)
-      (effects (font (size 1.27 1.27)) (justify left))
-    )
-    (property "Footprint" "Resistor_SMD:R_0402_1005Metric" (id 2) (at 321.31 238.76 0)
-      (effects (font (size 1.27 1.27)) hide)
-    )
-    (property "Datasheet" "~" (id 3) (at 321.31 238.76 0)
-      (effects (font (size 1.27 1.27)) hide)
-    )
-    (pin "1")
-    (pin "2")
-  )
   (symbol (lib_id "Device:Crystal_Small") (at 95.25 119.38 270) (unit 1)
     (in_bom yes) (on_board yes)
@@
     (pin "2")
   )
-  (symbol (lib_id "Device:C_Small") (at 170.18 262.89 0) (unit 1)
-    (in_bom yes) (on_board yes)
-    (property "Reference" "C73" (id 0) (at 172.72 261.62 0)
-      (effects (font (size 1.27 1.27)) (justify left))
-    )
-    (property "Value" "2n2" (id 1) (at 172.72 264.16 0)
-      (effects (font (size 1.27 1.27)) (justify left))
-    )
-    (property "Footprint" "Capacitor_SMD:C_0402_1005Metric" (id 2) (at 170.18 262.89 0)
-      (effects (font (size 1.27 1.27)) hide)
-    )
-    (property "Datasheet" "~" (id 3) (at 170.18 262.89 0)
-      (effects (font (size 1.27 1.27)) hide)
-    )
-    (pin "1")
-    (pin "2")
-  )
   (symbol (lib_id "Device:C_Small") (at 177.8 -2.54 0) (unit 1)
     (in_bom yes) (on_board yes)
@@
       (effects (font (size 1.27 1.27)) hide)
     )
-    (pin "1")
-    (pin "2")
-  )
-  (symbol (lib_id "Device:C_Small") (at 328.93 238.76 0) (unit 1)
-    (in_bom yes) (on_board yes)
-    (property "Reference" "C72" (id 0) (at 331.47 237.49 0)
-      (effects (font (size 1.27 1.27)) (justify left))
-    )
-    (property "Value" "2n2" (id 1) (at 331.47 240.03 0)
-      (effects (font (size 1.27 1.27)) (justify left))
-    )
-    (property "Footprint" "Capacitor_SMD:C_0402_1005Metric" (id 2) (at 328.93 238.76 0)
-      (effects (font (size 1.27 1.27)) hide)
-    )
-    (property "Datasheet" "~" (id 3) (at 328.93 238.76 0)
-      (effects (font (size 1.27 1.27)) hide)
-    )
